Commit message: new simulation

File: simulation_ws/src/cortador_description/urdf/cortador.xacro (robot description, xacro)
@@ -207,6 +207,6 @@
     <parent link="odom_link"/>
     <axis xyz="0 1 0" rpy="0 0 0"/>
-    <limit effort="100" velocity="100"/>
-    <joint_properties damping="0.0" friction="0.0"/>
+    <limit effort="10000" velocity="10000"/>
+    <joint_properties damping="1.0" friction="1.0"/>
   </joint>
   <joint type="continuous" name="right_wheel_hinge">
@@ -215,6 +215,6 @@
     <parent link="odom_link"/>
     <axis xyz="0 1 0" rpy="0 0 0"/>
-    <limit effort="100" velocity="100"/>
-    <joint_properties damping="0.0" friction="0.0"/>
+    <limit effort="10000" velocity="10000"/>
+    <joint_properties damping="1.0" friction="1.0"/>
   </joint>
  </robot>

Commit message: new simulation files

File: simulation_ws/src/cortador_description/urdf/cortador.xacro (robot description, xacro)
@@ -97,4 +97,16 @@
     <child link="odom_link"/>
   </joint>
+  <link name="sensor_link_right">
+    <xacro:sensor_link_macro l="${l_camera}"/>
+  </link>
+  <joint name="sensor_joint_right" type="fixed">
+    <xacro:sensor_joint_macro x="0" y="${-y_chassis/2}" z="${z_chassis/2}" l="${l_camera}" parent_link="chassis" child_link="sensor_link_right" a="0" b="0" c="-1.57"/>
+  </joint>
+   <link name="sensor_link_left">
+    <xacro:sensor_link_macro l="${l_camera}"/>
+  </link>
+  <joint name="sensor_joint_left" type="fixed">
+    <xacro:sensor_joint_macro x="0" y="${y_chassis/2}" z="${z_chassis/2}" l="${l_camera}" parent_link="chassis" child_link="sensor_link_left" a="0" b="0" c="1.57"/>
+  </joint>
   <!-- Chlorophyllsensors -->
 <!--<xacro:if value="${$(arg prefix) == 1}">-->
@@ -103,5 +115,5 @@
 	</link>
 	<joint name="camera_joint_mid" type="fixed">
-		<xacro:sensor_joint_macro x="${x_chassis/2 + l_camera/2}" y="0" z="${-z_chassis/2 + l_camera/2}" l="${l_camera}" parent_link="chassis" child_link="camera_link_mid"/>
+		<xacro:sensor_joint_macro x="${x_chassis/2 + l_camera/2}" y="0" z="${-z_chassis/2 + l_camera/2}" l="${l_camera}" parent_link="chassis" child_link="camera_link_mid" a="1.57" b="0" c="0"/>
 	</joint>
   <!--</xacro:if>-->
